File: matrix.kicad_sch (KiCad schematic)
At the start: 28 parts

Commit message: Added keys
Parts:
- added D15, D16, D17, D18, D19, D20, D21, D22, D23, D24, D25, D26, D27, D28, D29, D30, D31, D32, D33, D34, D35, D36, D37, D38, D39, D40, D41, D42, D43, D44, D45, D46, D47, D48, D49, D50, D51, D52, D53, D54, D55, D56, D57, D58, D59, D60, D61, D62: D, symbol Simulation_SPICE:DIODE
- added K15: TAB, symbol Switch:SW_Push
- added K16: Q, symbol Switch:SW_Push
- added K17: W, symbol Switch:SW_Push
- added K18: E, symbol Switch:SW_Push
- added K19: R, symbol Switch:SW_Push
- added K20: T, symbol Switch:SW_Push
- added K21: Y, symbol Switch:SW_Push
- added K22: U, symbol Switch:SW_Push
- added K23: I, symbol Switch:SW_Push
- added K24: O, symbol Switch:SW_Push
- added K25: P, symbol Switch:SW_Push
- added K26: [{, symbol Switch:SW_Push
- added K27: ]}, symbol Switch:SW_Push
- added K28: BSPC, symbol Switch:SW_Push
- added K29: CPLK, symbol Switch:SW_Push
- added K30: A, symbol Switch:SW_Push
- added K31: S, symbol Switch:SW_Push
- added K32: D, symbol Switch:SW_Push
- added K33: F, symbol Switch:SW_Push
- added K34: G, symbol Switch:SW_Push
- added K35: H, symbol Switch:SW_Push
- added K36: J, symbol Switch:SW_Push
- added K37: K, symbol Switch:SW_Push
- added K38: L, symbol Switch:SW_Push
- added K39: ;:, symbol Switch:SW_Push
- added K40: '", symbol Switch:SW_Push
- added K41: \|, symbol Switch:SW_Push
- added K42: ENTER, symbol Switch:SW_Push
- added K43: LSHIFT, symbol Switch:SW_Push
- added K44: Z, symbol Switch:SW_Push
- added K45: X, symbol Switch:SW_Push
- added K46: C, symbol Switch:SW_Push
- added K47: V, symbol Switch:SW_Push
- added K48: B, symbol Switch:SW_Push
- added K49: N, symbol Switch:SW_Push
- added K50: M, symbol Switch:SW_Push
- added K51: ,<, symbol Switch:SW_Push
- added K52: .>, symbol Switch:SW_Push
- added K53: /?, symbol Switch:SW_Push
- added K54: RSHIFT, symbol Switch:SW_Push
- added K55: FN1, symbol Switch:SW_Push
- added K56: LCTRL, symbol Switch:SW_Push
- added K57: LWIN, symbol Switch:SW_Push
- added K58: LALT, symbol Switch:SW_Push
- added K59: SPACE, symbol Switch:SW_Push
- added K60: RALT, symbol Switch:SW_Push
- added K61: RWIN, symbol Switch:SW_Push
- added K62: RCTRL, symbol Switch:SW_Push
- K1: renamed from K?; value SW_Push -> ESC
- K10: renamed from K?; value SW_Push -> #9
- K11: renamed from K?; value SW_Push -> #0
- K12: renamed from K?; value SW_Push -> -_
- K13: renamed from K?; value SW_Push -> =+
- K14: renamed from K?; value SW_Push -> \|
- K2: renamed from K?; value SW_Push -> #1
- K3: renamed from K?; value SW_Push -> #2
- K4: renamed from K?; value SW_Push -> #3
- K5: renamed from K?; value SW_Push -> #4
- K6: renamed from K?; value SW_Push -> #5
- K7: renamed from K?; value SW_Push -> #6
- K8: renamed from K?; value SW_Push -> #7
- K9: renamed from K?; value SW_Push -> #8
- gave numbers to parts that had none: 14
Connections:
- net row0: now reaches D1.2 (K), D10.2 (K), D11.2 (K), D12.2 (K), D13.2 (K), D14.2 (K), D2.2 (K), D3.2 (K), D4.2 (K), D5.2 (K), D6.2 (K), D7.2 (K), D8.2 (K), D9.2 (K)
- net col8: now reaches K9.2
- net col8: now also K23.2, K37.2, K51.2
- net col10: now reaches K11.2
- net col10: now also K25.2, K39.2, K53.2, K60.2
- net col7: now reaches K8.2
- net col7: now also K22.2, K36.2, K50.2
- net col6: now reaches K7.2
- net col6: now also K21.2, K35.2, K49.2, K59.2
- net col5: now reaches K6.2
- net col5: now also K20.2, K34.2, K48.2
- net col4: now reaches K5.2
- net col4: now also K19.2, K33.2, K47.2
- net col1: now reaches K2.2
- net col1: now also K16.2, K30.2, K44.2, K57.2
- net col9: now reaches K10.2
- net col9: now also K24.2, K38.2, K52.2
- net col0: now reaches K1.2
- net col0: now also K15.2, K29.2, K43.2, K56.2
- net col11: now reaches K12.2
- net col11: now also K26.2, K40.2, K54.2, K61.2
- net col3: now reaches K4.2
- net col3: now also K18.2, K32.2, K46.2
- net col13: now reaches K14.2
- net col13: now also K28.2, K42.2, K55.2, K62.2
- net col12: now reaches K13.2
- net col12: now also K27.2, K41.2
- net col2: now reaches K3.2
- net col2: now also K17.2, K31.2, K45.2, K58.2
- new net: D28.1 (A), K28.1
- new net: D26.1 (A), K26.1
- new net: D51.1 (A), K51.1
- new net: D16.1 (A), K16.1
- new net: D44.1 (A), K44.1
- new net: D50.1 (A), K50.1
- new net: D18.1 (A), K18.1
- new net: D46.1 (A), K46.1
- new net: D15.1 (A), K15.1
- new net: D32.1 (A), K32.1
- new net: D52.1 (A), K52.1
- new net: D29.1 (A), K29.1
- new net: D47.1 (A), K47.1
- new net: D56.1 (A), K56.1
- new net: D34.1 (A), K34.1
- new net: D39.1 (A), K39.1
- new net: D40.1 (A), K40.1
- new net: D30.1 (A), K30.1
- new net: D23.1 (A), K23.1
- new net: D41.1 (A), K41.1
- new net: D27.1 (A), K27.1
- new net: D25.1 (A), K25.1
- new net: D36.1 (A), K36.1
- new net: D43.1 (A), K43.1
- new net: D37.1 (A), K37.1
- new net: D19.1 (A), K19.1
- new net: D55.1 (A), K55.1
- new net: D17.1 (A), K17.1
- new net: D59.1 (A), K59.1
- new net: D58.1 (A), K58.1
- new net: D33.1 (A), K33.1
- new net: D57.1 (A), K57.1
- new net: D53.1 (A), K53.1
- new net: D48.1 (A), K48.1
- new net: D24.1 (A), K24.1
- new net: D60.1 (A), K60.1
- new net: D21.1 (A), K21.1
- new net: D49.1 (A), K49.1
- new net: D22.1 (A), K22.1
- new net: D20.1 (A), K20.1
- new net: D45.1 (A), K45.1
- new net: D35.1 (A), K35.1
- new net: D54.1 (A), K54.1
- new net: D62.1 (A), K62.1
- new net: D31.1 (A), K31.1
- new net: D38.1 (A), K38.1
- new net: D42.1 (A), K42.1
- new net: D61.1 (A), K61.1
- new net row1: D15.2 (K), D16.2 (K), D17.2 (K), D18.2 (K), D19.2 (K), D20.2 (K), D21.2 (K), D22.2 (K), D23.2 (K), D24.2 (K), D25.2 (K), D26.2 (K), D27.2 (K), D28.2 (K)
- new net row2: D29.2 (K), D30.2 (K), D31.2 (K), D32.2 (K), D33.2 (K), D34.2 (K), D35.2 (K), D36.2 (K), D37.2 (K), D38.2 (K), D39.2 (K), D40.2 (K), D41.2 (K), D42.2 (K)
- new net row3: D43.2 (K), D44.2 (K), D45.2 (K), D46.2 (K), D47.2 (K), D48.2 (K), D49.2 (K), D50.2 (K), D51.2 (K), D52.2 (K), D53.2 (K), D54.2 (K), D55.2 (K)
- new net row4: D56.2 (K), D57.2 (K), D58.2 (K), D59.2 (K), D60.2 (K), D61.2 (K), D62.2 (K)
Other:
- moved on the sheet: D1, D10, D11, D12, D13, D14, D2, D3, D4, D5, D6, D7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
