File: matrix.kicad_sch (KiCad schematic)
At the start: 124 parts, among them K1 ESC, K10 #9, K11 #0, K12 -_, K13 =+, K14 \|, K15 TAB, K16 Q, K17 W, K18 E, K19 R, K2 #1, K20 T, K21 Y, K22 U, K23 I, K24 O, K25 P, K26 [{, K27 ]}, K28 BSPC, K29 CPLK, K3 #2, K30 A, K31 S, K32 D, K33 F, K34 G, K35 H, K36 J, K37 K, K38 L, K39 ;:, K4 #3, K40 '", K41 \|, K42 ENTER, K43 LSHIFT, K44 Z, K45 X, K46 C, K47 V, K48 B, K49 N, K5 #4, K50 M, K51 ,<, K52 .>, K53 /?, K54 RSHIFT, K55 FN1, K56 LCTRL, K57 LWIN, K58 LALT, K59 SPACE, K6 #5, K60 RALT, K61 RWIN, K62 RCTRL, K7 #6, K8 #7, K9 #8

Commit message: added footprints
Parts:
- D1, D10, D11, D12, D13, D14, D15, D16, D17, D18, D19, D2, D20, D21, D22, D23, D24, D25, D26, D27, D28, D29, D3, D30, D31, D32, D33, D34, D35, D36, D37, D38, D39, D4, D40, D41, D42, D43, D44, D45, D46, D47, D48, D49, D5, D50, D51, D52, D53, D54, D55, D56, D57, D58, D59, D6, D60, D61, D62, D7, D8, D9: footprint (none) -> Diode_SMD:D_SOD-123
- K1, K10, K11, K12, K13, K14, K16, K17, K18, K19, K2, K20, K21, K22, K23, K24, K25, K26, K27, K3, K30, K31, K32, K33, K34, K35, K36, K37, K38, K39, K4, K40, K41, K44, K45, K46, K47, K48, K49, K5, K50, K51, K52, K53, K55, K57, K6, K61, K7, K8, K9: footprint (none) -> MX_Alps_Hybrid:MX-1U
- K15, K28, K56, K58, K60, K62: footprint (none) -> MX_Alps_Hybrid:MX-1.5U
- K29, K54: footprint (none) -> MX_Alps_Hybrid:MX-1.75U
- K42, K43: footprint (none) -> MX_Alps_Hybrid:MX-2.25U
- K59: footprint (none) -> MX_Alps_Hybrid:MX-7U

Commit message: created pcb w/o traces
Parts:
- K41: value \| -> DEL
- K59: footprint MX_Alps_Hybrid:MX-7U -> MX_Alps_Hybrid:MX-7U-ReversedStabilizers
Changed lines of the file:
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@@
     (in_bom yes) (on_board yes)
     (property "Reference" "K41" (id 0) (at 229.87 69.85 0))
-    (property "Value" "\\|" (id 1) (at 229.87 68.58 0)
+    (property "Value" "DEL" (id 1) (at 229.87 68.58 0)
       (effects (font (size 1.27 1.27)) hide)
     )
@@
       (effects (font (size 1.27 1.27)) hide)
     )
-    (property "Footprint" "MX_Alps_Hybrid:MX-7U" (id 2) (at 138.43 96.52 0)
-      (effects (font (size 1.27 1.27)) hide)
-    )
+    (property "Footprint" "MX_Alps_Hybrid:MX-7U-ReversedStabilizers" (id 2) (at 138.43 96.52 0)
+      (effects (font (size 1.27 1.27)) hide)
+    )

Commit message: pre final
Parts:
- K1: footprint MX_Alps_Hybrid:MX-1U -> MX_Hotswap:MX-Hotswap-1U
Changed lines of the file:
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@@
       (effects (font (size 1.27 1.27)) hide)
     )
-    (property "Footprint" "MX_Alps_Hybrid:MX-1U" (id 2) (at 46.99 40.64 0)
+    (property "Footprint" "MX_Hotswap:MX-Hotswap-1U" (id 2) (at 46.99 40.64 0)
       (effects (font (size 1.27 1.27)) hide)
     )
