File: jr60-pcb.kicad_pcb (KiCad board)
At the start: 2 copper layers, 285.8 x 99.3 mm, 145 parts, among them J1 AVR-ISP-6, K1 ESC, K10 #9, K11 #0, K12 -_, K13 =+, K14 \|, K15 TAB, K16 Q, K17 W, K18 E, K19 R, K2 #1, K20 T, K21 Y, K22 U, K23 I, K24 O, K25 P, K26 [{, K27 ]}, K28 BSPC, K29 CPLK, K3 #2, K30 A, K31 S, K32 D, K33 F, K34 G, K35 H, K36 J, K37 K, K38 L, K39 ;:, K4 #3, K40 '", K41 DEL, K42 ENTER, K43 LSHIFT, K44 Z, K45 X, K46 C, K47 V, K48 B, K49 N, K5 #4, K50 M, K51 ,<, K52 .>, K53 /?, K54 RSHIFT, K55 FN1, K56 LCTRL, K57 LWIN, K58 LALT, K59 SPACE, K6 #5, K60 RALT, K61 RWIN, K62 RCTRL, K7 #6, K8 #7, K9 #8, SW1 SW_Push, U1 ATmega32U4-A, U2 PRTR5V0U2X, X1 XTAL

Commit message: started column tracing
Routing:
- net col13: track 0.00 -> 103.7 mm
- net col1: track 0.00 -> 102.9 mm
- net col2: track 0.00 -> 100.1 mm
- net col11: track 0.00 -> 97.7 mm
- net col6: track 0.00 -> 92.1 mm
- net col10: track 0.00 -> 89.5 mm
- net col0: track 0.00 -> 84.3 mm
- net col12: track 0.00 -> 76.3 mm
- net col3: track 0.00 -> 71.7 mm
- net col4: track 0.00 -> 71.7 mm
- net col9: track 0.00 -> 70.7 mm
- net col8: track 0.00 -> 70.5 mm
- net col5: track 0.00 -> 70.5 mm
- net col7: track 0.00 -> 70.5 mm

Commit message: added all traces
Parts:
- moved J1 90.8 mm to (228.1, 108.4), turned to 0 degrees
- moved C7 2.92 mm to (205.9, 111.1)
- moved C8 2.92 mm to (205.9, 108.0)
- moved C2 2.51 mm to (196.1, 104.0)
- moved C1 1.34 mm to (191.8, 117.1)
- moved F1 1.12 mm to (42.1, 38.9)
- turned D1 to -90 degrees
- turned D10 to -90 degrees
- turned D11 to -90 degrees
- turned D12 to -90 degrees
- turned D13 to -90 degrees
- turned D14 to -90 degrees
- turned D15 to -90 degrees
- turned D16 to -90 degrees
- turned D17 to -90 degrees
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Connections:
- U1 pad 36: col6 -> row4
- U1 pad 38: row1 -> col6
- U1 pad 39: row4 -> row1
Routing:
- net GND: track 0.00 -> 405.3 mm, vias 0 -> 9
- net +5V: track 0.00 -> 370.0 mm, vias 0 -> 12
- net row2: track 0.00 -> 358.4 mm, vias 0 -> 6
- net row1: track 0.00 -> 351.9 mm, vias 0 -> 6
- net row0: track 0.00 -> 342.6 mm, vias 0 -> 4
- net row3: track 0.00 -> 295.2 mm, vias 0 -> 4
- net row4: track 0.00 -> 280.9 mm, vias 0 -> 2
- net D+: track 0.00 -> 202.2 mm
- net D-: track 0.00 -> 199.1 mm
- net col0: track 84.3 -> 275.8 mm, vias 0 -> 1
- net col12: track 76.3 -> 253.8 mm, vias 0 -> 1
- net col13: track 103.7 -> 242.5 mm, vias 0 -> 1
- net col1: track 102.9 -> 233.1 mm, vias 0 -> 3
- net col2: track 100.1 -> 204.8 mm, vias 0 -> 3
- net col3: track 71.7 -> 170.7 mm, vias 0 -> 3
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- added copper zone on B.Cu, net GND
- added copper zone on F.Cu, net GND
