File: jr60-pcb.kicad_pcb (KiCad board)
At the start: 2 copper layers, 285.8 x 99.3 mm, 145 parts, among them J1 AVR-ISP-6, K1 ESC, K10 #9, K11 #0, K12 -_, K13 =+, K14 \|, K15 TAB, K16 Q, K17 W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

Commit message: close to finish - at least I think
Parts:
- added G***: LOGO, Logos:Beard, F.Cu at (121.5, 108.7)
Other:
- board text added: "JR60 REV 0.1 Designed by Jöran Rieß"
